Commit message: Revert "Adding obstacle and moving bot"
This reverts commit 9ee5cf289a4d6900d7fe78d42bff4cd93412ab52.

File: description/robot.urdf.xacro (robot description, xacro)
@@ -2,4 +2,3 @@
 <robot xmlns:xacro="http://www.ros.org/wiki/xacro"  name="robot">
     <xacro:include filename="robot_core.xacro" />
-    <xacro:include filename="gazebo_control.xacro"/>
 </robot>

File: description/robot_core.xacro (robot description, xacro)
@@ -2,8 +2,8 @@
 <robot xmlns:xacro="http://www.ros.org/wiki/xacro" >
     <xacro:include filename="inertial_macros.xacro"/>
-    <material name="white">
+    <material name ="white">
         <color rgba="1 1 1 1" />
     </material>
-    <material name="orange">
+    <material name ="orange">
         <color rgba="1 0.3 0.1 1"/>
     </material>
@@ -14,8 +14,8 @@
         <color rgba="0 0 0 1"/>
     </material>
-    <!-- BASE LINK -->
+    <!-- BASE LINK-->
     <link name="base_link">
     </link>
-    <!-- CHASSIS LINK -->
+    <!-- CHASSIS LINK-->
     <joint name="chassis_joint" type="fixed">
         <parent link="base_link"/>
@@ -38,15 +38,12 @@
         </collision>
         <xacro:inertial_box mass="0.5" x="0.3" y="0.3" z="0.15">
-            <origin xyz="0.15 0 0.075" rpy="0 0 0"/>
+            <origin xyz=" 0.15 0 0.075" rpy="0 0 0"/>
         </xacro:inertial_box>
     </link>
-    <gazebo reference="chassis">
-        <material>Gazebo/White</material>
-    </gazebo>
-    <!-- LEFT WHEEL LINK -->
+    <!-- LEFT WHEEL LINK-->
     <joint name="left_wheel_joint" type="continuous">
         <parent link="base_link"/>
         <child link="left_wheel"/>
-        <origin xyz="0 0.175 0" rpy="-${pi/2} 0 0" />
+        <origin xyz="0 0.175 0" rpy="-${pi/2} 0 0"/> <!-- translation first, then rotation-->
         <axis xyz="0 0 1"/>
     </joint>
@@ -67,12 +64,9 @@
         </xacro:inertial_cylinder>
     </link>
-    <gazebo reference="left_wheel">
-        <material>Gazebo/Blue</material>
-    </gazebo>
-    <!-- RIGHT WHEEL LINK -->
+    <!--RIGHT WHEEL LINK-->
     <joint name="right_wheel_joint" type="continuous">
         <parent link="base_link"/>
         <child link="right_wheel"/>
-        <origin xyz="0 -0.175 0" rpy="${pi/2} 0 0" />
+        <origin xyz="0 -0.175 0" rpy="${pi/2} 0 0"/>
         <axis xyz="0 0 -1"/>
     </joint>
@@ -93,10 +87,7 @@
         </xacro:inertial_cylinder>
     </link>
-    <gazebo reference="right_wheel">
-        <material>Gazebo/Blue</material>
-    </gazebo>
-    <!-- CASTER WHEEL LINK -->
+    <!--CASTER WHEEL LINK-->
     <joint name="caster_wheel_joint" type="fixed">
-        <parent link="chassis"/>
+        <parent link='chassis'/>
         <child link="caster_wheel"/>
         <origin xyz="0.24 0 0"/>
@@ -105,5 +96,5 @@
         <visual>
             <geometry>
-                <sphere radius="0.05"/>
+                <sphere  radius="0.05"/>
             </geometry>
             <material name="black"/>
@@ -111,5 +102,5 @@
         <collision>
             <geometry>
-                <sphere radius="0.05"/>
+                <sphere  radius="0.05"/>
             </geometry>
         </collision>
@@ -118,8 +109,3 @@
         </xacro:inertial_sphere>
     </link>
-    <gazebo reference="caster_wheel">
-        <material>Gazebo/Black</material>
-        <mu1 value="0.001"/>
-        <mu2 value="0.001"/>
-    </gazebo>
 </robot>
